File: Hammond Arduino Base.kicad_pcb (KiCad board)
At the start: 2 copper layers, 120.4 x 100.1 mm, 86 parts, among them J1 SCI, J10 D8, J11 D7, J12 D6, J13 D5, J14 D4, J15 D3, J16 D2, J17 D1, J18 D0, J19 D14, J2 SDA, J20 D15, J21 D16, J22 D17, J23 D18, J24 D19, J25 D20, J26 D21, J27 5V, J28 5V, J29 D22, J3 AREF, J30 D23, J31 D24, J32 D25, J33 D26, J34 D27, J35 D28, J36 D29, J37 D30, J38 D31, J39 D32, J4 Gnd, J40 D33, J41 D34, J42 D35, J43 D36, J44 D37, J45 D38, J46 D39, J47 D40, J48 D41, J49 D42, J5 D13, J50 D43, J51 D44, J52 D45, J53 D46, J54 D47, J55 D48, J56 D49, J57 D50, J58 D51, J59 D52, J6 D12, J60 D53, J61 Gnd, J62 Gnd, J63 N/C, J64 IOREF, J65 RESET, J66 3.3V, J67 5V, J68 Gnd, J69 Gnd, J7 D11, J70 Vin, J71 A0, J72 A1, J73 A2, J74 A3, J75 A4, J76 A5, J77 A6, J78 A7, J79 A8, J8 D10, J80 A9, J81 A10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

Commit message: Add files via upload
Parts:
- renumbered J28 to J27, J27 to J28, J61 to J4, J4 to J61, J68 to J62, J62 to J68
Other:
- board text added: "Hammond 1455N1202 enclosure dimensions"
